Commit message: edit realsense and zed camera OBJ files their origin  and corresponding modeling direction
Also reflect changes in URDF

File: airo_models/cameras/realsense/d435/d435.urdf (robot description, URDF)
Before this commit: robot d435, 3 links, 2 joints
Links:
- removed link rgb_hole
- added link tripod_hole
- link d435_link: mass 0.175 -> 0.072; geometry collision box size=0.09 0.025 0.025; visual mesh filename=d435.obj scale=0.1 0.1 0.1
Joints:
- removed joint d435_link_2_rgb_hole
- added joint pose_of_tripod_hole_in_eye: type fixed, parent d435_link, child tripod_hole, origin xyz=-0.0325 -0.0125 -0.016 rpy=0 0 0
- joint base_link_2_d435_link: origin xyz=0 0 0.00 rpy=0 -1.57 1.57 -> xyz=0 0 0.00 rpy=0 0 0

File: airo_models/cameras/zed2i/zed2i.urdf (robot description, URDF)
Before this commit: robot zed2i, 2 links, 1 joints
Links:
- added link right_eye
- link zed_link: geometry collision box size=0.175 0.043 0.0373; visual mesh filename=zed2i.obj scale=0.1 0.1 0.1
Joints:
- added joint pose_of_right_eye_in_left_eye: type fixed, parent zed_link, child right_eye, origin xyz=-0.12 0 0 rpy=0 0 0
- joint base_link_2_zed_link: origin xyz=0 0 0.00 rpy=0 -1.57 -1.57 -> xyz=0 0 0.00 rpy=0 0 0

Commit message: d435i camera: change mesh origin and orientation so we can mount directly from camera calibration matrix

File: airo_models/cameras/realsense/d435/d435.urdf (robot description, URDF)
Before this commit: robot d435, 3 links, 2 joints
Joints:
- joint pose_of_tripod_hole_in_eye: origin xyz=-0.0325 -0.0125 -0.016 rpy=0 0 0 -> xyz=0.0325 0.0125 -0.016 rpy=0 0 0
