Commit message: schunk gripper: add collision box around cable plug

File: airo_models/grippers/schunk_egk40/urdf/schunk_egk40.urdf (robot description, URDF)
Before this commit: robot Schunk_EGK40_MB_M_B, 3 links, 2 joints
Links:
- link base_link: geometry collision box size=0.04 0.04 0.04; collision box size=0.117 0.068 0.0835
