Commit message: schunk magneto gripper: add mounting plate, pcb mounting plate and corresponding collision meshes

File: airo_models/grippers/schunk_egk40_magneto/schunk_egk40_magneto.urdf (robot description, URDF)
Before this commit: robot schunk_egk40_magneto, 5 links, 4 joints
Links:
- added link base_link_gripper, mass 1.02; collision box size=0.04 0.04 0.04; collision box size=0.117 0.068 0.0835
- added link camera_mount_plate; collision box size=0.117 0.068 0.0035; visual box size=0.117 0.068 0.0035
- added link pcb_mount_plate; collision box size=0.02 0.068 0.0835; visual box size=0.02 0.068 0.0835
- link base_link: mass 1.02 -> None; geometry collision box size=0.117 0.068 0.015; visual box size=0.117 0.068 0.015
Joints:
- added joint base_link_gripper_joint: type fixed, parent camera_mount_plate, child base_link_gripper
- added joint base_link_to_camera_mount_plate: type fixed, parent base_link, child camera_mount_plate
- added joint base_link_to_pcb_mount_plate: type fixed, parent base_link, child pcb_mount_plate, origin xyz=-0.0685 0 0.04175
- joint left_finger_mount_joint: parent base_link -> base_link_gripper
- joint right_finger_mount_joint: parent base_link -> base_link_gripper
