Commit message: Split base_link's geometry into a distinct adapter_plate link
base_link previously carried a 15mm-thick box directly, collocated at
the same origin as camera_mount_plate and base_link_gripper (all
three overlapped at z=0 instead of stacking in series). Give base_link
its own explicit adapter_plate child link (1cm thick) and chain the
gripper stack physically in series: base_link -> adapter_plate ->
camera_mount_plate -> base_link_gripper, with each link's origin
offset by its parent's thickness so the plates sit front-to-back
rather than overlapping.

This adds 13.5mm (10mm adapter_plate + 3.5mm camera_mount_plate) of
real standoff between tool0 and base_link_gripper that was previously
implicit/absorbed into base_link_gripper's own collision box. Anything
downstream that measures an offset from schunk_base_link/tool0 to the
gripper's TCP (e.g. realman-grasping's build_curobo_robot.py
TCP_OFFSET_Z) should be re-checked against this new stack-up.

File: airo_models/grippers/schunk_egk40_magneto/schunk_egk40_magneto.urdf (robot description, URDF)
Before this commit: robot schunk_egk40_magneto, 8 links, 7 joints
Links:
- added link adapter_plate; collision box size=0.117 0.068 0.01; visual box size=0.117 0.068 0.01
- link base_link: geometry 
Joints:
- removed joint base_link_to_camera_mount_plate
- added joint adapter_plate_to_camera_mount_plate: type fixed, parent adapter_plate, child camera_mount_plate, origin xyz=0 0 0.01
- added joint base_link_to_adapter_plate: type fixed, parent base_link, child adapter_plate
- joint base_link_gripper_joint: origin (none) -> xyz=0 0 0.0035

Commit message: Add a tcp link at the fingertips' contact face
New fixed "tcp" link, child of base_link_gripper, at z=0.1405 m
(0.0835 finger-mount height + 0.057 fingertip local z-extent, read
off magneto_finger.obj's flat tip face). The two finger mounts are
point-symmetric about x=0,y=0, so each fingertip's local x/y offset
cancels exactly in the average regardless of gripper opening -- only
the z (reach) term survives, making this frame's x/y independent of
the prismatic joint values.

This is a much more physically grounded TCP definition than
downstream consumers' previous ad-hoc offsets measured from
schunk_base_link/tool0 (e.g. realman-grasping's TCP_OFFSET_Z=0.0835,
which effectively placed the TCP inside the gripper body rather than
at the fingertips).

File: airo_models/grippers/schunk_egk40_magneto/schunk_egk40_magneto.urdf (robot description, URDF)
Before this commit: robot schunk_egk40_magneto, 9 links, 8 joints
Links:
- added link tcp
Joints:
- added joint base_link_gripper_to_tcp: type fixed, parent base_link_gripper, child tcp, origin xyz=0 0 0.1405 rpy=0 0 0

Commit message: improve fingertip collision box

File: airo_models/grippers/schunk_egk40_magneto/schunk_egk40_magneto.urdf (robot description, URDF)
Before this commit: robot schunk_egk40_magneto, 10 links, 9 joints
Links:
- link left_magneto_finger: geometry collision box size=0.025 0.025 0.057; visual mesh filename=../fingertips/meshes/magneto_finger.obj
- link right_magneto_finger: geometry collision box size=0.025 0.025 0.057; visual mesh filename=../fingertips/meshes/magneto_finger.obj
Joints:
- joint left_finger_mount_joint: limit lower=-0 upper=0.05 effort=10 velocity=0.1 -> lower=0 upper=0.04 effort=10 velocity=0.1; mimic (none) -> joint=right_finger_mount_joint multiplier=-1 offset=0; origin xyz=-0.0155 -0.01711 0.0835 rpy=0 0 0 -> xyz=-0.0135 -0.01711 0.0835 rpy=0 0 0
- joint right_finger_mount_joint: limit lower=-0.05 upper=0 effort=10 velocity=0.1 -> lower=-0.04 upper=0 effort=10 velocity=0.1; origin xyz=0.0155 0.01711 0.0835 rpy=0 0 0 -> xyz=0.0135 0.01711 0.0835 rpy=0 0 0
- joint right_finger_mount_to_tip: origin xyz=0 0 0 rpy=0 0 0 -> xyz=0.0 0 0 rpy=0 0 0

Commit message: use exact stroke width

File: airo_models/grippers/schunk_egk40_magneto/schunk_egk40_magneto.urdf (robot description, URDF)
Before this commit: robot schunk_egk40_magneto, 10 links, 9 joints
Joints:
- joint left_finger_mount_joint: limit lower=0 upper=0.04 effort=10 velocity=0.1 -> lower=0 upper=0.0415 effort=10 velocity=0.1; origin xyz=-0.0135 -0.01711 0.0835 rpy=0 0 0 -> xyz=-0.014 -0.01711 0.0835 rpy=0 0 0
- joint right_finger_mount_joint: limit lower=-0.04 upper=0 effort=10 velocity=0.1 -> lower=-0.0415 upper=0 effort=10 velocity=0.1; origin xyz=0.0135 0.01711 0.0835 rpy=0 0 0 -> xyz=0.014 0.01711 0.0835 rpy=0 0 0

Commit message: improve URDF of Schunk + airo fingertips (#24)
* Split base_link's geometry into a distinct adapter_plate link

base_link previously carried a 15mm-thick box directly, collocated at
the same origin as camera_mount_plate and base_link_gripper (all
three overlapped at z=0 instead of stacking in series). Give base_link
its own explicit adapter_plate child link (1cm thick) and chain the
gripper stack physically in series: base_link -> adapter_plate ->
camera_mount_plate -> base_link_gripper, with each link's origin
offset by its parent's thickness so the plates sit front-to-back
rather than overlapping.

This adds 13.5mm (10mm adapter_plate + 3.5mm camera_mount_plate) of
real standoff between tool0 and base_link_gripper that was previously
implicit/absorbed into base_link_gripper's own collision box. Anything
downstream that measures an offset from schunk_base_link/tool0 to the
gripper's TCP (e.g. realman-grasping's build_curobo_robot.py
TCP_OFFSET_Z) should be re-checked against this new stack-up.

* Add a tcp link at the fingertips' contact face

New fixed "tcp" link, child of base_link_gripper, at z=0.1405 m
(0.0835 finger-mount height + 0.057 fingertip local z-extent, read
off magneto_finger.obj's flat tip face). The two finger mounts are
point-symmetric about x=0,y=0, so each fingertip's local x/y offset
cancels exactly in the average regardless of gripper opening -- only
the z (reach) term survives, making this frame's x/y independent of
the prismatic joint values.

This is a much more physically grounded TCP definition than
downstream consumers' previous ad-hoc offsets measured from
schunk_base_link/tool0 (e.g. realman-grasping's TCP_OFFSET_Z=0.0835,
which effectively placed the TCP inside the gripper body rather than
at the fingertips).

* improve fingertip collision box

* use exact stroke width

* add readme for EGK-magneto model

File: airo_models/grippers/schunk_egk40_magneto/schunk_egk40_magneto.urdf (robot description, URDF)
Before this commit: robot schunk_egk40_magneto, 8 links, 7 joints
Links:
- added link adapter_plate; collision box size=0.117 0.068 0.01; visual box size=0.117 0.068 0.01
- added link tcp
- link base_link: geometry 
- link left_magneto_finger: geometry collision box size=0.025 0.025 0.057; visual mesh filename=../fingertips/meshes/magneto_finger.obj
- link right_magneto_finger: geometry collision box size=0.025 0.025 0.057; visual mesh filename=../fingertips/meshes/magneto_finger.obj
Joints:
- removed joint base_link_to_camera_mount_plate
- added joint adapter_plate_to_camera_mount_plate: type fixed, parent adapter_plate, child camera_mount_plate, origin xyz=0 0 0.01
- added joint base_link_gripper_to_tcp: type fixed, parent base_link_gripper, child tcp, origin xyz=0 0 0.1405 rpy=0 0 0
- added joint base_link_to_adapter_plate: type fixed, parent base_link, child adapter_plate
- joint base_link_gripper_joint: origin (none) -> xyz=0 0 0.0035
- joint left_finger_mount_joint: limit lower=-0 upper=0.05 effort=10 velocity=0.1 -> lower=0 upper=0.0415 effort=10 velocity=0.1; mimic (none) -> joint=right_finger_mount_joint multiplier=-1 offset=0; origin xyz=-0.0155 -0.01711 0.0835 rpy=0 0 0 -> xyz=-0.014 -0.01711 0.0835 rpy=0 0 0
- joint right_finger_mount_joint: limit lower=-0.05 upper=0 effort=10 velocity=0.1 -> lower=-0.0415 upper=0 effort=10 velocity=0.1; origin xyz=0.0155 0.01711 0.0835 rpy=0 0 0 -> xyz=0.014 0.01711 0.0835 rpy=0 0 0
- joint right_finger_mount_to_tip: origin xyz=0 0 0 rpy=0 0 0 -> xyz=0.0 0 0 rpy=0 0 0
