Commit message: Update collision boxes for KELO bricks

File: airo_models/mobile_platforms/kelo_robile/urdf/battery_brick.urdf (robot description, URDF)
Before this commit: robot battery_brick, 4 links, 3 joints
Links:
- link lid_link: geometry collision box size=0.233 0.233 0.24; visual mesh filename=../meshes/lid.obj scale=1 1 1

File: airo_models/mobile_platforms/kelo_robile/urdf/cpu_brick.urdf (robot description, URDF)
Before this commit: robot cpu_brick, 4 links, 3 joints
Links:
- link lid_link: geometry collision box size=0.233 0.233 0.24; visual mesh filename=../meshes/lid.obj scale=1 1 1

File: airo_models/mobile_platforms/kelo_robile/urdf/wheel_brick.urdf (robot description, URDF)
Before this commit: robot wheel_brick, 5 links, 4 joints
Links:
- link pivot_link: geometry collision box size=0.233 0.233 0.24; visual mesh filename=../meshes/kelo_drive_base.obj scale=1 1 1
