Commit message: Use relative paths for URDF to mesh

File: airo_models/arms/crx10ial/crx10ial.urdf (robot description, URDF)
Before this commit: robot fanuc_crx10ial, 10 links, 9 joints
Links:
- link base_link: geometry collision mesh filename=collision/base_link.stl; visual mesh filename=visual/base_link.stl
- link link_1: geometry collision mesh filename=collision/link_1.stl; visual mesh filename=visual/link_1.stl
- link link_2: geometry collision mesh filename=collision/link_2.stl; visual mesh filename=visual/link_2.stl
- link link_3: geometry collision mesh filename=collision/link_3.stl; visual mesh filename=visual/link_3.stl
- link link_4: geometry collision mesh filename=collision/link_4.stl; visual mesh filename=visual/link_4.stl
- link link_5: geometry collision mesh filename=collision/link_5.stl; visual mesh filename=visual/link_5.stl
- link link_6: geometry collision mesh filename=collision/link_6.stl; visual mesh filename=visual/link_6.stl

Commit message: Update STL -> OBJ in urdf

File: airo_models/arms/crx10ial/crx10ial.urdf (robot description, URDF)
Before this commit: robot fanuc_crx10ial, 10 links, 9 joints
Links:
- link base_link: geometry collision mesh filename=collision/base_link.obj; visual mesh filename=visual/base_link.obj
- link link_1: geometry collision mesh filename=collision/link_1.obj; visual mesh filename=visual/link_1.obj
- link link_2: geometry collision mesh filename=collision/link_2.obj; visual mesh filename=visual/link_2.obj
- link link_3: geometry collision mesh filename=collision/link_3.obj; visual mesh filename=visual/link_3.obj
- link link_4: geometry collision mesh filename=collision/link_4.obj; visual mesh filename=visual/link_4.obj
- link link_5: geometry collision mesh filename=collision/link_5.obj; visual mesh filename=visual/link_5.obj
- link link_6: geometry collision mesh filename=collision/link_6.obj; visual mesh filename=visual/link_6.obj
