Commit message: Add hull decimation and part cap to convex collision script
Expose CoACD --max-convex-hull (default 8) and --max-ch-vertex (default 64,
with decimate=True) and raise the default --threshold to 0.1. Regenerate the
RM75-6F convex variant: hulls now capped at 64 vertices (was up to 3800),
making whole-robot collision queries ~8x faster than before and now faster
than the raw-mesh collision model.

Co-authored-by: Copilot <223556219+Copilot@users.noreply.github.com>

File: airo_models/arms/rm75_6f/rm75_6f_convex_collision.urdf (robot description, URDF)
Before this commit: robot RM75-6F, 10 links, 9 joints
Links:
- link base_link: geometry collision mesh filename=collision_convex/base_link_collision_0_part_0.obj; collision mesh filename=collision_convex/base_link_collision_0_part_1.obj
- link link_1: geometry collision mesh filename=collision_convex/link_1_collision_0_part_0.obj; collision mesh filename=collision_convex/link_1_collision_0_part_1.obj
- link link_2: geometry collision mesh filename=collision_convex/link_2_collision_0_part_0.obj; collision mesh filename=collision_convex/link_2_collision_0_part_1.obj
- link link_3: geometry collision mesh filename=collision_convex/link_3_collision_0_part_0.obj; collision mesh filename=collision_convex/link_3_collision_0_part_1.obj
- link link_4: geometry collision mesh filename=collision_convex/link_4_collision_0_part_0.obj; collision mesh filename=collision_convex/link_4_collision_0_part_1.obj
- link link_5: geometry collision mesh filename=collision_convex/link_5_collision_0_part_0.obj; collision mesh filename=collision_convex/link_5_collision_0_part_1.obj
- link link_6: geometry collision mesh filename=collision_convex/link_6_collision_0_part_0.obj; collision mesh filename=collision_convex/link_6_collision_0_part_1.obj
- link link_7: geometry collision mesh filename=collision_convex/link_7_collision_0_part_0.obj; collision mesh filename=collision_convex/link_7_collision_0_part_1.obj
