Commit message: urdf STL to OBJ for Drake

File: airo_models/arms/rm75_6f/rm75_6f.urdf (robot description, URDF)
Before this commit: robot RM75-6F, 10 links, 9 joints
Links:
- link base_link: geometry collision mesh filename=collision/base_link_collision_0_part_0.obj; collision mesh filename=collision/base_link_collision_0_part_1.obj
- link link_1: geometry collision mesh filename=collision/link_1_collision_0_part_0.obj; collision mesh filename=collision/link_1_collision_0_part_1.obj
- link link_2: geometry collision mesh filename=collision/link_2_collision_0_part_0.obj; collision mesh filename=collision/link_2_collision_0_part_1.obj
- link link_3: geometry collision mesh filename=collision/link_3_collision_0_part_0.obj; collision mesh filename=collision/link_3_collision_0_part_1.obj
- link link_4: geometry collision mesh filename=collision/link_4_collision_0_part_0.obj; collision mesh filename=collision/link_4_collision_0_part_1.obj
- link link_5: geometry collision mesh filename=collision/link_5_collision_0_part_0.obj; collision mesh filename=collision/link_5_collision_0_part_1.obj
- link link_6: geometry collision mesh filename=collision/link_6_collision_0_part_0.obj; collision mesh filename=collision/link_6_collision_0_part_1.obj
- link link_7: geometry collision mesh filename=collision/link_7_collision_0_part_0.obj; collision mesh filename=collision/link_7_collision_0_part_1.obj

File: airo_models/arms/rm75_6f/rm75_6f_primitives.urdf (robot description, URDF)
Before this commit: robot RM75-6F, 10 links, 9 joints
Links:
- link base_link: geometry collision cylinder length=0.13850000514891364 radius=0.05714995227754116; visual mesh filename=visual/base_link.obj
- link link_1: geometry collision cylinder length=0.14250008016824722 radius=0.054514115676283836; visual mesh filename=visual/link_1.obj
- link link_2: geometry collision cylinder length=0.19299999997019768 radius=0.04099998623132706; visual mesh filename=visual/link_2.obj
- link link_3: geometry collision cylinder length=0.1375000737607479 radius=0.05100001394748688; visual mesh filename=visual/link_3.obj
- link link_4: geometry collision cylinder length=0.16249999776482582 radius=0.037000044248998165; visual mesh filename=visual/link_4.obj
- link link_5: geometry collision cylinder length=0.11000007204711437 radius=0.04149998631328344; visual mesh filename=visual/link_5.obj
- link link_6: geometry collision cylinder length=0.1434748787432909 radius=0.034249961376190186; visual mesh filename=visual/link_6.obj
- link link_7: geometry collision cylinder length=0.05750000899195662 radius=0.03316052071750164; visual mesh filename=visual/link_7.obj
