Commit message: Add base/tool0 frames and primitive collision model to RM75-6F
Add ROS-Industrial base and tool0 frames to rm75_6f.urdf as fixed joints
with identity transforms; per RealMan's official URDFs/driver, the
manufacturer base and tool frames match base_link and link_7 with no
z-rotation. Regenerate the convex-collision variant to include them.

Add scripts/generate_primitive_collision_meshes.py, which fits one bounding
cylinder per collision mesh (axis = longest extent, overridable via
--axis-map). Apply it to produce rm75_6f_primitives.urdf (link_2/4/6
horizontal, others vertical) and register it as 'rm75_6f_primitives'.

Co-authored-by: Copilot <223556219+Copilot@users.noreply.github.com>

File: airo_models/arms/rm75_6f/rm75_6f.urdf (robot description, URDF)
Before this commit: robot RM75-6F, 8 links, 7 joints
Links:
- added link base
- added link tool0
Joints:
- added joint base_link-base: type fixed, parent base_link, child base, origin xyz=0 0 0 rpy=0 0 0
- added joint link_7-tool0: type fixed, parent link_7, child tool0, origin xyz=0 0 0 rpy=0 0 0

File: airo_models/arms/rm75_6f/rm75_6f_primitives.urdf (robot description, URDF)
Before this commit: robot RM75-6F, 10 links, 9 joints
Links:
- link base_link: geometry collision cylinder length=0.13850000514891364 radius=0.05714995227754116; visual mesh filename=visual/base_link.STL
- link link_1: geometry collision cylinder length=0.14250008016824722 radius=0.054514115676283836; visual mesh filename=visual/link_1.STL
- link link_2: geometry collision cylinder length=0.19299999997019768 radius=0.04099998623132706; visual mesh filename=visual/link_2.STL
- link link_3: geometry collision cylinder length=0.1375000737607479 radius=0.05100001394748688; visual mesh filename=visual/link_3.STL
- link link_4: geometry collision cylinder length=0.16249999776482582 radius=0.037000044248998165; visual mesh filename=visual/link_4.STL
- link link_5: geometry collision cylinder length=0.11000007204711437 radius=0.04149998631328344; visual mesh filename=visual/link_5.STL
- link link_6: geometry collision cylinder length=0.1434748787432909 radius=0.034249961376190186; visual mesh filename=visual/link_6.STL
- link link_7: geometry collision cylinder length=0.05750000899195662 radius=0.03316052071750164; visual mesh filename=visual/link_7.STL

Commit message: Make convex hulls the default RM75-6F collision; drop raw-mesh variant
The rm75_6f model now uses the CoACD convex decomposition as its collision
geometry (folder renamed collision_convex/ -> collision/), and the separate
rm75_6f_convex_collision model and the raw-mesh collision/ STLs are removed.
Both collision-generation scripts now derive collision geometry from each
link's visual mesh instead of a pre-existing collision mesh. README and the
model registry are updated to the two-variant layout (rm75_6f default,
rm75_6f_primitives).

Co-authored-by: Copilot <223556219+Copilot@users.noreply.github.com>

File: airo_models/arms/rm75_6f/rm75_6f.urdf (robot description, URDF)
Before this commit: robot RM75-6F, 10 links, 9 joints
Links:
- link base_link: geometry collision mesh filename=collision/base_link_collision_0_part_0.obj; collision mesh filename=collision/base_link_collision_0_part_1.obj
- link link_1: geometry collision mesh filename=collision/link_1_collision_0_part_0.obj; collision mesh filename=collision/link_1_collision_0_part_1.obj
- link link_2: geometry collision mesh filename=collision/link_2_collision_0_part_0.obj; collision mesh filename=collision/link_2_collision_0_part_1.obj
- link link_3: geometry collision mesh filename=collision/link_3_collision_0_part_0.obj; collision mesh filename=collision/link_3_collision_0_part_1.obj
- link link_4: geometry collision mesh filename=collision/link_4_collision_0_part_0.obj; collision mesh filename=collision/link_4_collision_0_part_1.obj
- link link_5: geometry collision mesh filename=collision/link_5_collision_0_part_0.obj; collision mesh filename=collision/link_5_collision_0_part_1.obj
- link link_6: geometry collision mesh filename=collision/link_6_collision_0_part_0.obj; collision mesh filename=collision/link_6_collision_0_part_1.obj
- link link_7: geometry collision mesh filename=collision/link_7_collision_0_part_0.obj; collision mesh filename=collision/link_7_collision_0_part_1.obj

Commit message: Fix rm75_6f J7 joint limit: 6.28 -> 6.2832 (exact 2π / ±360°)
Co-authored-by: Copilot <223556219+Copilot@users.noreply.github.com>

File: airo_models/arms/rm75_6f/rm75_6f.urdf (robot description, URDF)
Before this commit: robot RM75-6F, 10 links, 9 joints
Joints:
- joint joint_7: limit lower=-6.28 upper=6.28 effort=10 velocity=3.14 -> lower=-6.2832 upper=6.2832 effort=10 velocity=3.14

File: airo_models/arms/rm75_6f/rm75_6f_primitives.urdf (robot description, URDF)
Before this commit: robot RM75-6F, 10 links, 9 joints
Joints:
- joint joint_7: limit lower=-6.28 upper=6.28 effort=10 velocity=3.14 -> lower=-6.2832 upper=6.2832 effort=10 velocity=3.14

Commit message: Fix rm75_6f: use RM75-6FB meshes/kinematics (d7 = 161.2 mm)
The folder literally named RM75-6F in RealManRobot/rm_models uses
joint_7 = 172.5 mm, which has no corresponding official parameter set
and is likely a stale or different flange revision.

The official RealMan developer docs define d7 = 161.2 mm for the
RM75-6F (Six-Axis Force) robot, which maps to the RM75-6FB folder
(joint_7 = 161.2 mm). FK cross-checked against three poses recorded
from the robot's control UI: <1 mm position error, <0.001 rad
orientation error.

Changes:
- Replace link_7 visual mesh (STL + OBJ) with RM75-6FB version
- Replace link_7 CoACD collision parts with RM75-6FB version
- Update joint_7 origin in rm75_6f.urdf: 0.1725 -> 0.1612 m
- Regenerate rm75_6f_primitives.urdf (link_7 cylinder: 57.5 -> 46.0 mm)
- Remove temporary rm75_6fb model (no longer needed)
- Tighten FK test tolerance from 15 mm to 1 mm
- Document the RM75-6F vs RM75-6FB naming cross-check in README

Co-authored-by: Copilot <223556219+Copilot@users.noreply.github.com>

File: airo_models/arms/rm75_6f/rm75_6f.urdf (robot description, URDF)
Before this commit: robot RM75-6F, 10 links, 9 joints
Joints:
- joint joint_7: origin xyz=0 -0.1725 0 rpy=1.5708 0 0 -> xyz=0 -0.1612 0 rpy=1.5708 0 0

File: airo_models/arms/rm75_6f/rm75_6f_primitives.urdf (robot description, URDF)
Before this commit: robot RM75-6F, 10 links, 9 joints
Links:
- link base_link: geometry collision cylinder length=0.13850001 radius=0.05714995; visual mesh filename=visual/base_link.obj
- link link_1: geometry collision cylinder length=0.14250008 radius=0.054514115; visual mesh filename=visual/link_1.obj
- link link_2: geometry collision cylinder length=0.193 radius=0.040999985; visual mesh filename=visual/link_2.obj
- link link_3: geometry collision cylinder length=0.13750007 radius=0.051000015; visual mesh filename=visual/link_3.obj
- link link_4: geometry collision cylinder length=0.1625 radius=0.03700004; visual mesh filename=visual/link_4.obj
- link link_5: geometry collision cylinder length=0.11000006999999999 radius=0.04149999; visual mesh filename=visual/link_5.obj
- link link_6: geometry collision cylinder length=0.14347487 radius=0.034249959999999996; visual mesh filename=visual/link_6.obj
- link link_7: geometry collision cylinder length=0.046 radius=0.03065; visual mesh filename=visual/link_7.obj
Joints:
- joint joint_7: origin xyz=0 -0.1725 0 rpy=1.5708 0 0 -> xyz=0 -0.1612 0 rpy=1.5708 0 0
